File: hardware/schematic/v1.0/SIG_COND/SIG_COND.kicad_sch (KiCad schematic)
At the start: 12 parts, among them J1 Conn_Coaxial, K1 G6K-2F-RF, K3 G6K-2F-Y-5V, Q1 AO3400A, Q3 AO3400A, U1 PE43705

Commit message: chore: 更新原理图和配置文件
Parts:
- added J2: USB_C_Receptacle_USB2.0_16P, Connector_USB:USB_C_Receptacle_GCT_USB4105-xx-A_16P_TopMnt_Horizontal, symbol Connector:USB_C_Receptacle_USB2.0_16P
- added U2: SN65LVDS20, Package_SO:SOIC-8-1EP_3.9x4.9mm_P1.27mm_EP2.29x3mm, symbol Counter:SN65LVDS20
- added U3: ADCMP573, Package_CSP:LFCSP-16-1EP_3x3mm_P0.5mm_EP1.3x1.3mm, symbol Counter:ADCMP573
Connections:
- net RF_OUT is gone; now on an unnamed net: K1.6
- net SMA_IN1 is gone; now on net SMA_IN: J1.1 (In)
- net SMA_IN: now reaches K1.3
- new net: J2.A1 (GND), J2.A12 (GND), J2.B1 (GND), J2.B12 (GND)
- new net: J2.A4 (VBUS), J2.A9 (VBUS), J2.B4 (VBUS), J2.B9 (VBUS)
Other:
- moved on the sheet: D3, K3, Q3, R7, U1

Commit message: chore: 更新 KiCad 原理图相关配置
Parts:
- added J4, J5: Conn_Coaxial, Connector_Coaxial:SMA_Amphenol_132289_EdgeMount, symbol Connector:Conn_Coaxial
- added U4: THS4303, Package_DFN_QFN:VQFN-16-1EP_3x3mm_P0.5mm_EP1.45x1.45mm, symbol Counter:THS4303
- J1: footprint Connector_Coaxial:SMA_Amphenol_132134_Vertical -> Connector_Coaxial:SMA_Amphenol_132289_EdgeMount
Connections:
- net GND: now also J4.2 (Ext), J5.2 (Ext)

Commit message: sch update
Parts:
- added C1: 1.7pF, symbol Device:C
- added C2: 15pF, symbol Device:C
- added C3, C5: 100nF, symbol Device:C
- added C4, C6: 10uF, symbol Device:C
- added R3: 100K, Resistor_SMD:R_0603_1608Metric, symbol Device:R
- added R4: 49.9 ±0.1%, Resistor_SMD:R_0603_1608Metric, symbol Device:R
- added U5: OPA659, Package_TO_SOT_SMD:TSOT-23-5, symbol Amplifier_Operational:OPA188xxDBV
- K3: value G6K-2F-Y-5V -> G6K-2F-RF
- R2: value 30 -> 900K
Connections:
- net +5V: now also C3.2, C4.2, U5.5 (V+)
- net GND: now also C2.2, C3.1, C4.1, C5.2, C6.2, R3.2
- net at R2.1: now also C1.1, C2.1, R3.1, U5.3 (+); no longer K1.4
- net at R2.2: now also K1.4, C1.2; no longer K1.5
- net ACDC1 renamed ACDC
- net SIG1 renamed Z0
- new net: K1.5, R4.2
- new net: R4.1, U5.1, U5.4 (-)
- new net -5V: C5.1, C6.1, U5.2 (V-)

Commit message: sch update
Parts:
- removed C1: 1.7pF, symbol Device:C
- removed C2: 15pF, symbol Device:C
- removed C3, C5: 100nF, symbol Device:C
- removed C4, C6: 10uF, symbol Device:C
- removed U1: PE43705, Package_DFN_QFN:QFN-32-1EP_5x5mm_P0.5mm_EP3.1x3.1mm, symbol Counter:PE43705
- removed U4: THS4303, Package_DFN_QFN:VQFN-16-1EP_3x3mm_P0.5mm_EP1.45x1.45mm, symbol Counter:THS4303
- removed U5: OPA659, Package_TO_SOT_SMD:TSOT-23-5, symbol Amplifier_Operational:OPA188xxDBV
- added C13: 18pF, symbol Device:C
- added C7: 1.7pF, symbol Device:C
- added C8: 15pF, symbol Device:C
- added R10, R11, R12: 10K, Resistor_SMD:R_0603_1608Metric, symbol Device:R
- added R6: 900K, Resistor_SMD:R_0603_1608Metric, symbol Device:R
- added R8: 100K, Resistor_SMD:R_0603_1608Metric, symbol Device:R
- added U1: LMH6518, Package_DFN_QFN:WQFN-16-1EP_4x4mm_P0.5mm_EP2.6x2.6mm_ThermalVias, symbol Counter:LMH6518
- R2: value 900K -> 15
- R3: value 100K -> 0
- R4: value 49.9 ±0.1% -> 30
Connections:
- net ACDC: now also R11.1; no longer Q3.1 (G)
- net GND: now also C8.2, R8.2; no longer R3.2
- net Z0: now also R10.1; no longer Q1.1 (G)
- net at R2.1, R3.1: now also K1.5
- net at K1.4, R2.2: now also R1.1, C13.2
- net at R4.2: now also K1.7; no longer K1.5
- net at K1.6: now also K3.3
- net at R4.1: now also K1.2
- net at K3.2: now also C7.2, R6.2
- net at K3.4: now also K3.5
- net at K3.7: now also C7.1, C8.1, R6.1, R8.1
- new net: C13.1, R3.2
- new net: Q1.1 (G), R10.2
- new net: Q3.1 (G), R11.2
- new net +3.3V: R12.2
- new net SCLK: U1.11 (SCLK)
- new net SDIO: U1.10 (SDIO)
- new net nCS: R12.1, U1.9 (nCS)
Other:
- note added: "Attenuator"
- moved on the sheet: D3, K3, Q3, R5, R7, U2, U3

Commit message: sch update
Parts:
- added R13, R14: 0, Resistor_SMD:R_0603_1608Metric, symbol Device:R
Connections:
- net GND: now also U1.17 (PAD), U1.5 (GND), U1.8 (GND)
- net VCM: now reaches U1.13 (VCM)
- net at U1.14 (-OUT): now also R14.1
- net at U1.15 (+OUT): now also R13.2
- no-connect marks 0 -> 3
