File: hardware/schematic/v1.0/Thunderscope_Rev5.3/FE_Channel.kicad_sch (KiCad schematic)
At the start: 105 parts, among them J1002_4 BNC, J3_4 UFL, J4_4 UFL, K1000_4 UD2-4.5NUN-L, K1001_4 UD2-4.5NUN-L, Q1002_4 DMN62D0UW, Q1003_4 DMN62D0UW, U1001_4 TMUX4053, U1008_4 LMH6518, U1009_4 BUF802, U1011_4 OPA140AIDBVR

Commit message: sch update
Parts:
- removed J3_4, J4_4: UFL, Thunderscope_Rev5:TE_2334884-1, symbol Thunderscope_Rev5:UFL Jack SMD
- added R52_5, R97_5: 0, Thunderscope_Rev5:GEN_R_0402, symbol Thunderscope_Rev5:RES 0 OHM 1/16W 0402
Connections:
- net at U1008_4.1 (AUX_P): now also R52_5.1
- net at U1008_4.2 (AUX_N): now also R97_5.1
- new net AUX_N: R97_5.2
- new net AUX_P: R52_5.2
- no-connect marks 4 -> 1
