File: hardware/schematic/v1.0/Thunderscope_Rev5.3/Thunderscope_Rev5.3.kicad_sch (KiCad schematic)
At the start: 16 parts

Commit message: sch update
Other:
- removed sheet ACQ and FE Voltage Regs
- removed sheet ADC
- removed sheet Clock Generator
- removed sheet FPGA
- removed sheet Front End Trim and Bias
- removed sheet TS-PCIe Components
- removed sheet TS-USB4 Components

Commit message: sch update
Other:
- added sheet ACQ and FE Voltage Regs (ACQ_FE_VREG.kicad_sch)
- added sheet ADC (ADC.kicad_sch)
- added sheet Clock Generator (PLL.kicad_sch)
- added sheet FPGA (FPGA.kicad_sch)
- added sheet Front End Trim and Bias (FE.kicad_sch)
- added sheet TS-PCIe Components (CON_PCIe_X4.kicad_sch)
- added sheet TS-USB4 Components (M2_KEY_M.kicad_sch)
