File: hardware/schematic/v1.0/Thunderscope_CH1_only/Thunderscope_Rev5.3.kicad_pcb (KiCad board)
At the start: 6 copper layers, 116 parts, among them J1 Conn_Coaxial, J3_1 UFL, J4_1 UFL, K1000_1 G6K-2F-RF, K1001_1 G6K-2F-RF, Q1002_1 DMN62D0UW, Q1003_1 DMN62D0UW, U1001_1 TMUX4053, U1008_1 LMH6518, U1009_1 BUF802, U1011_1 OPA140AIDBVR, U12_1 ADA4930-1YCPZ

Commit message: sch update
Parts:
- added C1043_2: 100nF, Thunderscope_Rev5:GEN_C_0402, F.Cu at (138.5, 63.8)
- added C104_2: 10nF, Thunderscope_Rev5:GEN_C_0402, F.Cu at (210.6, 57.4)
- added C104_3: 100pF, Thunderscope_Rev5:GEN_C_0402, F.Cu at (210.6, 59.5)
- added C104_4: 100pF, Thunderscope_Rev5:GEN_C_0402, F.Cu at (210.6, 61.6)
- added C104_5: 100nF, Thunderscope_Rev5:GEN_C_0402, F.Cu at (210.6, 63.7)
- added C104_6: 100nF, Thunderscope_Rev5:GEN_C_0402, F.Cu at (210.6, 65.9)
- added FB1000_2: 120@100MHZ, Thunderscope_Rev5:GEN_R_0402, F.Cu at (210.5, 68.0)
- added FB1000_3: 120@100MHZ, Thunderscope_Rev5:GEN_R_0402, F.Cu at (210.5, 70.0)
- added J2: Conn_Coaxial, Connector_Coaxial:SMA_Molex_73251-1153_EdgeMount_Horizontal, F.Cu at (159.3, 90.9)
- added J3: Conn_Coaxial, Connector_Coaxial:SMA_Molex_73251-1153_EdgeMount_Horizontal, F.Cu at (159.3, 106.8)
- added J4: Conn_Coaxial, Connector_Coaxial:SMA_Molex_73251-1153_EdgeMount_Horizontal, F.Cu at (205.8, 62.9)
- added J5: Conn_Coaxial, Connector_Coaxial:SMA_Molex_73251-1153_EdgeMount_Horizontal, F.Cu at (205.8, 76.1)
- added R136_2: 0, Thunderscope_Rev5:GEN_R_0402, F.Cu at (210.5, 72.1)
- added R136_3: 0, Thunderscope_Rev5:GEN_R_0402, F.Cu at (210.5, 74.2)
- added R136_4: 100, Thunderscope_Rev5:GEN_R_0402, F.Cu at (210.5, 76.3)
- added R137_10: 49.9, Thunderscope_Rev5:GEN_R_0402, F.Cu at (216.5, 74.2)
- added R137_2: 1.3K, Thunderscope_Rev5:GEN_R_0402, F.Cu at (213.5, 68.0)
- added R137_3: 499, Thunderscope_Rev5:GEN_R_0402, F.Cu at (213.5, 70.0)
- added R137_4: 127, Thunderscope_Rev5:GEN_R_0402, F.Cu at (213.5, 72.1)
- added R137_5: 82.5, Thunderscope_Rev5:GEN_R_0402, F.Cu at (213.5, 74.2)
- added R137_6: 127, Thunderscope_Rev5:GEN_R_0402, F.Cu at (213.5, 76.3)
- added R137_7: 82.5, Thunderscope_Rev5:GEN_R_0402, F.Cu at (216.5, 68.0)
- added R137_8: 0, Thunderscope_Rev5:GEN_R_0402, F.Cu at (216.5, 70.0)
- added R137_9: 49.9, Thunderscope_Rev5:GEN_R_0402, F.Cu at (216.5, 72.1)
- added R52_2: 0, Thunderscope_Rev5:GEN_R_0402, F.Cu at (197.4, 86.9)
- added R97_2: 0, Thunderscope_Rev5:GEN_R_0402, F.Cu at (197.4, 89.0)
- added U1: ADCMP573, Package_CSP:LFCSP-16-1EP_3x3mm_P0.5mm_EP1.3x1.3mm, F.Cu at (215.1, 59.0)
- added U2: SN65LVDS20, Package_SO:SOIC-8-1EP_3.9x4.9mm_P1.27mm_EP2.29x3mm, F.Cu at (213.3, 80.7)
- added U3: REF3012, Package_TO_SOT_SMD:SOT-23, F.Cu at (141.9, 62.9)
- moved R134_1 31.0 mm to (142.9, 72.2)
- moved R135_1 31.0 mm to (141.0, 72.2)
- moved C104_1 31.0 mm to (139.8, 77.4)
- moved R132_1 31.0 mm to (142.4, 70.8)
- moved R133_1 31.0 mm to (141.5, 70.8)
- moved R136_1 31.0 mm to (142.4, 77.8)
- moved R137_1 31.0 mm to (141.5, 77.8)
- moved C105_1 31.0 mm to (139.3, 73.8)
- moved C70_1 31.0 mm to (139.3, 75.7)
- moved R131_1 31.0 mm to (142.0, 69.4)
- moved U12_1 31.0 mm to (142.0, 74.8)
Connections:
- R136_1 pad 2: /ADC Driver 1/OUT_N -> Net-(J2-In)
- R137_1 pad 2: /ADC Driver 1/OUT_P -> Net-(J3-In)
- U1008_1 pad 1: unconnected-(U1008_1-AUX_P-Pad1) -> /AUX_P
- U1008_1 pad 16: unconnected-(U1008_1-AUX_VCM-Pad16) -> Net-(U1008_1-AUX_VCM)
- U1008_1 pad 2: unconnected-(U1008_1-AUX_N-Pad2) -> /AUX_N
Routing:
- net /CH1_N: track 63.6 -> 6.82 mm
- net /CH1_P: track 63.8 -> 7.25 mm
- net /ADC Driver 1/OUT_P: track 8.46 -> 0.00 mm
- net /ADC Driver 1/OUT_N: track 8.46 -> 0.00 mm
