File: hardware/schematic/v1.0/Thunderscope_CH1_only/Thunderscope_Rev5.3.kicad_pcb (KiCad board)
At the start: 6 copper layers, 145 parts, among them J1 Conn_Coaxial, J2 Conn_Coaxial, J3 Conn_Coaxial, J3_1 UFL, J4 Conn_Coaxial, J4_1 UFL, J5 Conn_Coaxial, K1000_1 G6K-2F-RF, K1001_1 G6K-2F-RF, Q1002_1 DMN62D0UW, Q1003_1 DMN62D0UW, U1 ADCMP573, U1001_1 TMUX4053, U1008_1 LMH6518, U1009_1 BUF802, U1011_1 OPA140AIDBVR, U12_1 ADA4930-1YCPZ, U2 SN65LVDS20, U3 REF3012

Commit message: sch and pcb update
Parts:
- C1036_1, C1037_1, C1038_1, C1039_1, C1040_1, C1043_2, FB1000_1, U3: moved to B.Cu
- moved C104_3 67.2 mm to (143.4, 59.5), turned to 90 degrees
- moved U1 66.4 mm to (148.9, 63.9)
- moved C104_4 65.1 mm to (145.5, 59.5), turned to 90 degrees
- moved R137_2 63.4 mm to (150.5, 60.7), turned to 90 degrees
- moved R137_7 63.2 mm to (153.5, 62.7), turned to -90 degrees
- moved C104_5 63.1 mm to (147.6, 59.5), turned to 90 degrees
- moved R137_6 62.9 mm to (152.0, 62.7), turned to 90 degrees
- moved R137_4 61.9 mm to (152.0, 65.1), turned to -90 degrees
- moved R97_2 61.8 mm to (141.3, 63.1)
- moved R137_5 60.7 mm to (153.5, 65.1), turned to 90 degrees
- moved R52_2 60.6 mm to (141.3, 64.1)
- moved R137_3 55.6 mm to (163.6, 45.6)
- moved FB1000_2 55.6 mm to (160.6, 43.5)
- moved U2 53.4 mm to (162.6, 64.1)
- moved C104_2 51.1 mm to (160.5, 67.7)
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Connections:
- net Net-(J2-In) renamed /ADC Driver 1/ADC_P
- net Net-(J3-In) renamed /ADC Driver 1/ADC_N
- C104_2 pad 1: Net-(U1-VCCO/VTT) -> Net-(U2-VBB)
- C104_3 pad 1: Net-(C104_3-Pad1) -> Net-(U1-VCCO/VTT)
- C104_4 pad 1: Net-(C104_3-Pad1) -> Net-(U1-VCCO/VTT)
- C104_5 pad 1: Net-(C104_3-Pad1) -> Net-(U1-VCCO/VTT)
- FB1000_2 pad 1: Net-(C104_3-Pad1) -> Net-(U1-VCCO/VTT)
- R137_3 pad 1: Net-(C104_3-Pad1) -> Net-(U1-VCCO/VTT)
- R137_4 pad 2: Net-(C104_3-Pad1) -> Net-(U1-VCCO/VTT)
- R137_6 pad 2: Net-(C104_3-Pad1) -> Net-(U1-VCCO/VTT)
- R52_2 pad 1: /AUX_P -> /CH1/AUX_R_P
- R52_2 pad 2: /AUX_P -> /RF_P
- R97_2 pad 1: /AUX_N -> /CH1/AUX_R_N
- R97_2 pad 2: /AUX_N -> /RF_N
- U1 pad 12: Net-(C104_3-Pad1) -> Net-(U1-VCCO/VTT)
- U1 pad 16: Net-(C104_3-Pad1) -> Net-(U1-VCCO/VTT)
- U1 pad 2: /AUX_P -> /RF_P
- U1 pad 3: /AUX_N -> /RF_N
- U1 pad 5: Net-(C104_3-Pad1) -> Net-(U1-VCCO/VTT)
- U1 pad 9: Net-(C104_3-Pad1) -> Net-(U1-VCCO/VTT)
- U1008_1 pad 1: /AUX_P -> /CH1/AUX_R_P
- U1008_1 pad 2: /AUX_N -> /CH1/AUX_R_N
- U2 pad 4: Net-(U1-VCCO/VTT) -> Net-(U2-VBB)
Routing:
- net /ADC Driver 1/ADC_N: track 0.00 -> 14.2 mm
- net /ADC Driver 1/ADC_P: track 0.00 -> 14.2 mm
- removed copper zone on F.Cu, net +5V
- removed copper zone on F.Cu, net /CH1/+VPGA
