File: hardware/schematic/v1.0/Thunderscope_CH1_only/ADC_Driver.kicad_sch (KiCad schematic)
At the start: 12 parts, among them U12_1 ADA4930-1YCPZ

Commit message: sch update
Parts:
- added C104_2: 10nF, Thunderscope_Rev5:GEN_C_0402, symbol Thunderscope_Rev5:CAP 1uF 25V X5R 0402
- added C104_3, C104_4: 100pF, Thunderscope_Rev5:GEN_C_0402, symbol Thunderscope_Rev5:CAP 1uF 25V X5R 0402
- added C104_5, C104_6: 100nF, Thunderscope_Rev5:GEN_C_0402, symbol Thunderscope_Rev5:CAP 1uF 25V X5R 0402
- added FB1000_2, FB1000_3: 120@100MHZ, Thunderscope_Rev5:GEN_R_0402, symbol Thunderscope_Rev5:FERRITE BEAD 120 OHM 0402
- added J2, J3, J4, J5: Conn_Coaxial, Connector_Coaxial:SMA_Molex_73251-1153_EdgeMount_Horizontal, symbol Connector:Conn_Coaxial
- added R136_2, R136_3, R137_8: 0, Thunderscope_Rev5:GEN_R_0402, symbol Thunderscope_Rev5:RES 4.99 OHM 1% 1/16W 0402
- added R136_4: 100, Thunderscope_Rev5:GEN_R_0402, symbol Thunderscope_Rev5:RES 4.99 OHM 1% 1/16W 0402
- added R137_10, R137_9: 49.9, Thunderscope_Rev5:GEN_R_0402, symbol Thunderscope_Rev5:RES 4.99 OHM 1% 1/16W 0402
- added R137_2: 1.3K, Thunderscope_Rev5:GEN_R_0402, symbol Thunderscope_Rev5:RES 4.99 OHM 1% 1/16W 0402
- added R137_3: 499, Thunderscope_Rev5:GEN_R_0402, symbol Thunderscope_Rev5:RES 4.99 OHM 1% 1/16W 0402
- added R137_4, R137_6: 127, Thunderscope_Rev5:GEN_R_0402, symbol Thunderscope_Rev5:RES 4.99 OHM 1% 1/16W 0402
- added R137_5, R137_7: 82.5, Thunderscope_Rev5:GEN_R_0402, symbol Thunderscope_Rev5:RES 4.99 OHM 1% 1/16W 0402
- added U1: ADCMP573, Package_CSP:LFCSP-16-1EP_3x3mm_P0.5mm_EP1.3x1.3mm, symbol Counter:ADCMP573
- added U2: SN65LVDS20, Package_SO:SOIC-8-1EP_3.9x4.9mm_P1.27mm_EP2.29x3mm, symbol Counter:SN65LVDS20
Connections:
- net +3V3_ACQ: now also FB1000_2.2, FB1000_3.2
- net GND: now also C104_2.2, C104_3.2, C104_4.2, C104_5.2, C104_6.1, J2.2 (Ext), J3.2 (Ext), J4.2 (Ext), J5.2 (Ext), R137_10.2, R137_2.2, R137_5.1, R137_7.1, R137_8.1, R137_9.1, U1.13 (GND), U1.15 (GND), U1.17 (PAD), U2.9 (GND)
- net OUT_N: no longer names the net of R136_1.2
- net OUT_N: now also J2.1 (In)
- net OUT_P: no longer names the net of R137_1.2
- net OUT_P: now also J3.1 (In)
- new net: R137_4.1, R137_5.2, U1.10 (nQ), U2.3 (B)
- new net: C104_3.1, C104_4.1, C104_5.1, FB1000_2.1, R137_3.1, R137_4.2, R137_6.2, U1.12 (VCCO), U1.16 (VCCI), U1.5 (VCCI), U1.9 (VCCO)
- new net: R137_3.2, U1.7 (LE)
- new net: R137_6.1, R137_7.2, U1.11 (Q), U2.2 (A)
- new net: R137_2.1, U1.14 (HYS)
- new net: C104_2.1, U1.8 (VCCO/VTT), U2.4 (VBB)
- new net: J4.1 (In), R136_2.2, R136_4.2, R137_9.2
- new net: R137_8.2, U2.5 (nEN)
- new net: R136_3.1, U2.6 (Z)
- new net: R136_2.1, U2.7 (Y)
- new net: C104_6.2, FB1000_3.1, U2.8 (VCC)
- new net: J5.1 (In), R136_3.2, R136_4.1, R137_10.1
- new net IN1_N: U1.3 (VN)
- new net IN1_P: U1.2 (VP)
- no-connect marks 0 -> 4
Other:
- moved on the sheet: C104_1, C105_1, C69_1, C70_1, R131_1, R132_1, R133_1, R134_1, R135_1, R136_1, R137_1, U12_1

Commit message: sch and pcb update
Connections:
- net at C104_3.1, C104_4.1, C104_5.1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: now also U1.8 (VCCO/VTT)
- net ADC_N: now reaches J3.1 (In), R137_1.2
- net ADC_P: now reaches J2.1 (In), R136_1.2
- net at C104_2.1, U2.4 (VBB): no longer U1.8 (VCCO/VTT)
Changed lines of the file:
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@@
+	)
+	(junction
+		(at 142.24 157.48)
+		(diameter 0)
+		(color 0 0 0 0)
 	)
 	(junction
@@
 	(junction
 		(at 130.81 38.1)
-		(diameter 0)
-		(color 0 0 0 0)
-	)
-	(junction
-		(at 172.72 142.24)
 		(diameter 0)
 		(color 0 0 0 0)
@@
 	(wire
 		(pts
+			(xy 128.27 157.48) (xy 142.24 157.48)
+		)
+		(stroke
+			(width 0)
+			(type default)
+		)
+	)
+	(wire
+		(pts
 			(xy 110.49 132.08) (xy 111.76 132.08)
 		)
@@
 	(wire
 		(pts
-			(xy 162.56 142.24) (xy 172.72 142.24)
-		)
-		(stroke
-			(width 0)
-			(type default)
-		)
-	)
-	(wire
-		(pts
 			(xy 143.51 83.82) (xy 143.51 86.36)
 		)
@@
 	(wire
 		(pts
+			(xy 142.24 157.48) (xy 142.24 163.83)
+		)
+		(stroke
+			(width 0)
+			(type default)
+		)
+	)
+	(wire
+		(pts
 			(xy 137.16 134.62) (xy 142.24 134.62)
 		)
@@
 	(wire
 		(pts
-			(xy 142.24 142.24) (xy 142.24 163.83)
+			(xy 142.24 142.24) (xy 142.24 157.48)
 		)
 		(stroke
@@
 	(wire
 		(pts
-			(xy 162.56 157.48) (xy 162.56 142.24)
-		)
-		(stroke
-			(width 0)
-			(type default)
-		)
-	)
-	(wire
-		(pts
 			(xy 143.51 58.42) (xy 146.05 58.42)
 		)
@@
 	(wire
 		(pts
-			(xy 128.27 157.48) (xy 162.56 157.48)
-		)
-		(stroke
-			(width 0)
-			(type default)
-		)
-	)
-	(wire
-		(pts
 			(xy 168.91 83.82) (xy 168.91 86.36)
 		)
@@
 		)
 	)
+	(label "ADC_P"
+		(at 189.23 63.5 180)
+		(effects
+			(font
+				(size 1.27 1.27)
+			)
+			(justify right bottom)
+		)
+	)
+	(label "ADC_N"
+		(at 189.23 68.58 180)
+		(effects
+			(font
+				(size 1.27 1.27)
+			)
+			(justify right bottom)
+		)
+	)
