File: hardware/schematic/v1.0/Thunderscope_CH1_only/Thunderscope_Rev5.3.kicad_sch (KiCad schematic)
At the start: 0 parts

Commit message: sch update
Other:
- sheet ADC Driver 1 ports: added IN1_N, IN1_P; removed OUT_N, OUT_P
- sheet CH1 ports: added AUX_N, AUX_P, VCM_AUX; removed none

Commit message: sch and pcb update
Changed lines of the file:
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@@
 		)
 	)
-	(label "AUX_P"
+	(label "RF_P"
 		(at 130.81 99.06 180)
 		(effects
@@
 		)
 	)
-	(label "AUX_N"
+	(label "RF_N"
 		(at 130.81 101.6 180)
 		(effects
