File: hardware/schematic/v1.0/Thunderscope_Rev5.3_CH1/External_IO.kicad_sch (KiCad schematic)
At the start: 7 parts, among them J1 Conn_01x03_Socket, J2 Conn_01x03_Socket, J3 Conn_02x06_Odd_Even

Commit message: sch and pcb update
Parts:
- J3: footprint Connector_PinSocket_1.27mm:PinSocket_2x06_P1.27mm_Vertical_SMD -> Connector_PinSocket_1.27mm:PinSocket_2x06_P1.27mm_Horizontal
Changed lines of the file:
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@@
+		)
+	)
+	(hierarchical_label "VCM"
+		(shape output)
+		(at 92.71 129.54 180)
+		(effects
+			(font
+				(size 1.27 1.27)
+			)
+			(justify right)
 		)
 	)
@@
 			)
 		)
-		(property "Footprint" "Connector_PinSocket_1.27mm:PinSocket_2x06_P1.27mm_Vertical_SMD"
+		(property "Footprint" "Connector_PinSocket_1.27mm:PinSocket_2x06_P1.27mm_Horizontal"
 			(at 165.1 139.7 0)
 			(hide yes)
