File: hardware/schematic/v1.0/Thunderscope_Rev5.3_CH1/Thunderscope_Rev5.3.kicad_pcb (KiCad board)
At the start: 6 copper layers, 53.7 x 23.1 mm, 104 parts, among them J1002_1 BNC, J3_1 UFL, J4_1 UFL, K1000_1 UD2-4.5NUN-L, K1001_1 UD2-4.5NUN-L, Q1002_1 DMN62D0UW, Q1003_1 DMN62D0UW, U1001_1 TMUX4053, U1008_1 LMH6518, U1009_1 BUF802, U1011_1 OPA140AIDBVR

Commit message: sch and pcb update
Parts:
- added J1: Conn_01x03_Socket, Connector_PinHeader_2.54mm:PinHeader_1x03_P2.54mm_Vertical, F.Cu at (92.7, 43.0)
- added J2: Conn_01x03_Socket, Connector_PinHeader_2.54mm:PinHeader_1x03_P2.54mm_Vertical, F.Cu at (134.8, 74.8)
- added J3: Conn_02x06_Odd_Even, Connector_PinSocket_1.27mm:PinSocket_2x06_P1.27mm_Vertical_SMD, B.Cu at (148.0, 65.5)
- added R52_8: 0, Thunderscope_Rev5:GEN_R_0402, F.Cu at (148.0, 52.9)
- added R97_8: 0, Thunderscope_Rev5:GEN_R_0402, F.Cu at (148.0, 54.9)
- added RF1: KH-IPEX-K501-29, JLCImport:KH-IPEX-K501-29, F.Cu at (141.5, 63.5)
- added RF2: KH-IPEX-K501-29, JLCImport:KH-IPEX-K501-29, F.Cu at (141.5, 69.1)
- added RF3: KH-IPEX-K501-29, JLCImport:KH-IPEX-K501-29, F.Cu at (147.4, 78.2)
- added RF4: KH-IPEX-K501-29, JLCImport:KH-IPEX-K501-29, F.Cu at (147.4, 73.8)
- K1000_1, K1001_1: value UD2-4.5NUN-L -> G6K-2F-RF
Connections:
- U1008_1 pad 1: unconnected-(U1008_1-AUX_P-Pad1) -> /CH1/AUX_R_P
- U1008_1 pad 2: unconnected-(U1008_1-AUX_N-Pad2) -> /CH1/AUX_R_N
Routing:
- net GND: track 55.9 -> 54.5 mm, vias 417 -> 414
- net +5V: track 15.3 -> 14.3 mm, vias 11 -> 9
- net +3V3_PGA: track 5.69 -> 4.77 mm, vias 4 -> 2
- net /DC_CPL_1: track 15.8 -> 16.6 mm, vias 1 -> 2
- net /PGA_SCLK: vias 1 -> 2
- net /PGA_CSn_1: vias 1 -> 2
- removed copper zone on F.Cu, net +3V3_PGA
Other:
- board size 53.7 x 23.1 mm -> 65 x 23.1 mm
- board text removed: "PGA LDO"

Commit message: sch and pcb update
Parts:
- removed J3_1, J4_1: UFL, Thunderscope_Rev5:TE_2334884-1
- C1037_1, C1040_1, FB1000_1: moved to B.Cu
- J3: footprint Connector_PinSocket_1.27mm:PinSocket_2x06_P1.27mm_Vertical_SMD -> Connector_PinSocket_1.27mm:PinSocket_2x06_P1.27mm_Horizontal
- moved R52_8 22.6 mm to (143.8, 75.0), turned to -90 degrees
- moved R97_8 20.4 mm to (144.8, 75.0), turned to -90 degrees
- moved J3 3.16 mm to (149.1, 62.6)
- moved FB1000_1 2.17 mm to (136.7, 63.4)
- moved C1040_1 2.11 mm to (137.8, 60.5), turned to 0 degrees
- moved C1037_1 1.67 mm to (133.3, 62.5), turned to 180 degrees
- moved RF3 0.56 mm to (147.4, 78.8)
- moved RF4 0.56 mm to (147.4, 73.3)
Connections:
- U1008_1 pad 16: unconnected-(U1008_1-AUX_VCM-Pad16) -> /VCM
Routing:
- net /CH1/AUX_R_N: track 0.00 -> 25.4 mm
- net /CH1/AUX_R_P: track 0.00 -> 24.7 mm
- net /CH1_AUX_P: track 0.00 -> 5.04 mm
- net /VCM: track 1.20 -> 4.85 mm, vias 1 -> 2
- net /CH1/+VPGA: track 0.05 -> 3.22 mm, vias 0 -> 2
- net /CH1_AUX_N: track 0.00 -> 2.98 mm
- net GND: track 54.5 -> 57.4 mm, vias 414 -> 416
- net /CH1_P: track 0.49 -> 3.28 mm
- net /CH1_N: track 0.49 -> 3.27 mm
- net +5V: track 14.3 -> 17.1 mm
- net /CH1/OUT_R_N: track 2.14 -> 1.44 mm, vias 1 -> 0
- net /CH1/OUT_R_P: track 2.12 -> 1.47 mm, vias 1 -> 0
