File: hardware/schematic/v1.0/Thunderscope_Rev5.3_CH1/Thunderscope_Rev5.3.kicad_sch (KiCad schematic)
At the start: 0 parts

Commit message: sch and pcb update
Other:
- added sheet IO (External_IO.kicad_sch)
- sheet CH1 ports: added AUX_N, AUX_P; removed none

Commit message: sch and pcb update
Other:
- sheet IO ports: added VCM; removed none
Changed lines of the file:
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@@
 	(wire
 		(pts
-			(xy 116.84 109.22) (xy 147.32 109.22)
-		)
-		(stroke
-			(width 0)
-			(type default)
-		)
-	)
-	(wire
-		(pts
-			(xy 116.84 106.68) (xy 147.32 106.68)
-		)
-		(stroke
-			(width 0)
-			(type default)
-		)
-	)
-	(wire
-		(pts
-			(xy 116.84 116.84) (xy 147.32 116.84)
-		)
-		(stroke
-			(width 0)
-			(type default)
-		)
-	)
-	(wire
-		(pts
-			(xy 116.84 119.38) (xy 147.32 119.38)
+			(xy 116.84 110.49) (xy 147.32 110.49)
+		)
+		(stroke
+			(width 0)
+			(type default)
+		)
+	)
+	(wire
+		(pts
+			(xy 116.84 107.95) (xy 147.32 107.95)
+		)
+		(stroke
+			(width 0)
+			(type default)
+		)
+	)
+	(wire
+		(pts
+			(xy 116.84 118.11) (xy 147.32 118.11)
+		)
+		(stroke
+			(width 0)
+			(type default)
+		)
+	)
+	(wire
+		(pts
+			(xy 116.84 120.65) (xy 147.32 120.65)
 		)
 		(stroke
@@
 	(wire
 		(pts
-			(xy 116.84 114.3) (xy 147.32 114.3)
+			(xy 116.84 115.57) (xy 147.32 115.57)
 		)
 		(stroke
@@
 	(wire
 		(pts
-			(xy 116.84 104.14) (xy 147.32 104.14)
-		)
-		(stroke
-			(width 0)
-			(type default)
-		)
-	)
-	(wire
-		(pts
-			(xy 116.84 99.06) (xy 129.54 99.06)
-		)
-		(stroke
-			(width 0)
-			(type default)
-		)
-	)
-	(wire
-		(pts
-			(xy 116.84 124.46) (xy 129.54 124.46)
+			(xy 116.84 105.41) (xy 147.32 105.41)
+		)
+		(stroke
+			(width 0)
+			(type default)
+		)
+	)
+	(wire
+		(pts
+			(xy 116.84 99.06) (xy 147.32 99.06)
+		)
+		(stroke
+			(width 0)
+			(type default)
+		)
+	)
+	(wire
+		(pts
+			(xy 116.84 125.73) (xy 129.54 125.73)
 		)
 		(stroke
@@
 	)
 	(label "PGA_SCLK"
-		(at 129.54 104.14 180)
+		(at 129.54 105.41 180)
 		(effects
 			(font
@@
 	)
 	(label "PGA_CSn_1"
-		(at 129.54 109.22 180)
+		(at 129.54 110.49 180)
 		(effects
 			(font
@@
 	)
 	(label "PGA_SDIO"
-		(at 129.54 106.68 180)
+		(at 129.54 107.95 180)
 		(effects
 			(font
@@
 	)
 	(label "ATTEN_1"
-		(at 129.54 116.84 180)
+		(at 129.54 118.11 180)
 		(effects
 			(font
@@
 	)
 	(label "TERM_1"
-		(at 129.54 114.3 180)
+		(at 129.54 115.57 180)
 		(effects
 			(font
@@
 	)
 	(label "DC_CPL_1"
-		(at 129.54 119.38 180)
+		(at 129.54 120.65 180)
 		(effects
 			(font
@@
 	)
 	(label "TRIM_1"
-		(at 129.54 124.46 180)
+		(at 129.54 125.73 180)
 		(effects
 			(font
@@
 		)
 		(pin "ATTEN" output
-			(at 147.32 116.84 180)
+			(at 147.32 118.11 180)
 			(effects
 				(font
@@
 		)
 		(pin "DC_CPL" output
-			(at 147.32 119.38 180)
+			(at 147.32 120.65 180)
 			(effects
 				(font
@@
 		)
 		(pin "TERM" output
-			(at 147.32 114.3 180)
+			(at 147.32 115.57 180)
 			(effects
 				(font
@@
 		)
 		(pin "PGA_SCLK" output
-			(at 147.32 104.14 180)
+			(at 147.32 105.41 180)
 			(effects
 				(font
@@
 		)
 		(pin "PGA_SDIO" output
-			(at 147.32 106.68 180)
+			(at 147.32 107.95 180)
 			(effects
 				(font
@@
 		)
 		(pin "PGA_CSn" output
-			(at 147.32 109.22 180)
+			(at 147.32 110.49 180)
+			(effects
+				(font
+					(size 1.27 1.27)
+				)
+				(justify left)
+			)
+		)
+		(pin "VCM" output
+			(at 147.32 99.06 180)
 			(effects
 				(font
@@
 	(sheet
 		(at 99.06 83.82)
-		(size 17.78 43.18)
+		(size 17.78 44.45)
 		(exclude_from_sim no)
 		(in_bom yes)
@@
 		)
 		(property "Sheetfile" "FE_Channel.kicad_sch"
-			(at 99.06 127.5846 0)
+			(at 99.06 128.8546 0)
 			(show_name no)
 			(do_not_autoplace no)
@@
 		)
 		(pin "TRIM" input
-			(at 116.84 124.46 0)
+			(at 116.84 125.73 0)
 			(effects
 				(font
@@
 		)
 		(pin "ATTEN" input
-			(at 116.84 116.84 0)
+			(at 116.84 118.11 0)
 			(effects
 				(font
@@
 		)
 		(pin "DC_CPL" input
-			(at 116.84 119.38 0)
+			(at 116.84 120.65 0)
 			(effects
 				(font
@@
 		)
 		(pin "PGA_CSn" input
-			(at 116.84 109.22 0)
+			(at 116.84 110.49 0)
 			(effects
 				(font
@@
 		)
 		(pin "PGA_SCLK" input
-			(at 116.84 104.14 0)
+			(at 116.84 105.41 0)
 			(effects
 				(font
@@
 		)
 		(pin "PGA_SDIO" input
-			(at 116.84 106.68 0)
+			(at 116.84 107.95 0)
 			(effects
 				(font
@@
 		)
 		(pin "TERM" input
-			(at 116.84 114.3 0)
-			(effects
-				(font
+			(at 116.84 115.57 0)
+			(effects
+				(font
